Commit message: 已经能正常开启导航并且完善了容器中缺乏的功能包

File: install/fishbot_description/share/fishbot_description/urdf/fishbot_base.urdf (robot description, URDF)
Before this commit: robot fishbot, 7 links, 6 joints
Links:
- link base_link: mass 0.2 -> None; geometry visual cylinder length=0.12 radius=0.10
- link caster_link: mass 0.02 -> None; geometry visual sphere radius=0.016
- link imu_link: mass 0.1 -> None; geometry visual box size=0.02 0.02 0.02
- link laser_link: mass 0.1 -> None; geometry visual cylinder length=0.02 radius=0.02
- link left_wheel_link: mass 0.2 -> None; geometry visual cylinder length=0.04 radius=0.032
- link right_wheel_link: mass 0.2 -> None; geometry visual cylinder length=0.04 radius=0.032
